Commit message: Modificando nome do diretório no marvin.urdf

File: ProjFinal/ros2_marvin/install/marvin_description/share/marvin_description/urdf/marvin.urdf (robot description, URDF)
Before this commit: robot robot_marvin_urdf, 8 links, 7 joints
Links:
- link base_link: geometry collision mesh filename=package://marvin_description/meshes/base_link.STL; visual mesh filename=package://marvin_description/meshes/base_link.STL
- link link_1: geometry collision mesh filename=package://marvin_description/meshes/link_1.STL; visual mesh filename=package://marvin_description/meshes/link_1.STL
- link link_22: geometry collision mesh filename=package://marvin_description/meshes/link_22.STL; visual mesh filename=package://marvin_description/meshes/link_22.STL
- link link_3: geometry collision mesh filename=package://marvin_description/meshes/link_3.STL; visual mesh filename=package://marvin_description/meshes/link_3.STL
- link link_4: geometry collision mesh filename=package://marvin_description/meshes/link_4.STL; visual mesh filename=package://marvin_description/meshes/link_4.STL
- link link_5: geometry collision mesh filename=package://marvin_description/meshes/link_5.STL; visual mesh filename=package://marvin_description/meshes/link_5.STL
- link link_6: geometry collision mesh filename=package://marvin_description/meshes/link_6.STL; visual mesh filename=package://marvin_description/meshes/link_6.STL
- link link_7: geometry collision mesh filename=package://marvin_description/meshes/link_7.STL; visual mesh filename=package://marvin_description/meshes/link_7.STL

File: ProjFinal/ros2_marvin/src/marvin_description/urdf/marvin.urdf (robot description, URDF)
Before this commit: robot marvin, 8 links, 7 joints
Links:
- link base_link: geometry collision mesh filename=package://marvin_description/meshes/base_link.STL; visual mesh filename=package://marvin_description/meshes/base_link.STL
- link link_1: geometry collision mesh filename=package://marvin_description/meshes/link_1.STL; visual mesh filename=package://marvin_description/meshes/link_1.STL
- link link_22: geometry collision mesh filename=package://marvin_description/meshes/link_22.STL; visual mesh filename=package://marvin_description/meshes/link_22.STL
- link link_3: geometry collision mesh filename=package://marvin_description/meshes/link_3.STL; visual mesh filename=package://marvin_description/meshes/link_3.STL
- link link_4: geometry collision mesh filename=package://marvin_description/meshes/link_4.STL; visual mesh filename=package://marvin_description/meshes/link_4.STL
- link link_5: geometry collision mesh filename=package://marvin_description/meshes/link_5.STL; visual mesh filename=package://marvin_description/meshes/link_5.STL
- link link_6: geometry collision mesh filename=package://marvin_description/meshes/link_6.STL; visual mesh filename=package://marvin_description/meshes/link_6.STL
- link link_7: geometry collision mesh filename=package://marvin_description/meshes/link_7.STL; visual mesh filename=package://marvin_description/meshes/link_7.STL

Commit message: Adicionando o pacote marvin_description ao marvin_bringup

File: ProjFinal/ros2_marvin/install/marvin_description/share/marvin_description/urdf/marvin.urdf (robot description, URDF)
Before this commit: robot marvin, 8 links, 7 joints
Joints:
- joint joint_1: axis 0 0 0 -> 0.0 0.0 0.0; limit lower=0 upper=3.142 effort=300 velocity=3 -> lower=0.0 upper=3.142 effort=300.0 velocity=3.0; origin xyz=0 0.405 0 rpy=0 -1.5708 0 -> xyz=0.0 0.405 0.0 rpy=0.0 -1.5708 0.0
- joint joint_2: axis 0 0 0 -> 0.0 0.0 0.0; limit lower=-1.57 upper=1.57 effort=200 velocity=3 -> lower=-1.57 upper=1.57 effort=200.0 velocity=3.0; origin xyz=0 0 0 rpy=0 0 0 -> xyz=0.0 0.0 0.0 rpy=0.0 0.0 0.0
- joint joint_3: axis 0 0 0 -> 0.0 0.0 0.0; limit lower=0 upper=3.142 effort=200 velocity=3 -> lower=0.0 upper=3.142 effort=200.0 velocity=3.0; origin xyz=0 0 0 rpy=0 0 0 -> xyz=0.0 0.0 0.0 rpy=0.0 0.0 0.0
- joint joint_4: axis 0 0 0 -> 0.0 0.0 0.0; limit lower=0 upper=-3.142 effort=200 velocity=3 -> lower=0.0 upper=-3.142 effort=200.0 velocity=3.0; origin xyz=0.05 -0.75 0 rpy=3.1416 0 -1.5708 -> xyz=0.05 -0.75 0.0 rpy=3.1416 0.0 -1.5708
- joint joint_5: axis 0 0 0 -> 0.0 0.0 0.0; limit lower=0 upper=3.142 effort=200 velocity=3 -> lower=0.0 upper=3.142 effort=200.0 velocity=3.0; origin xyz=0.002 0 0 rpy=0 0 0 -> xyz=0.002 0.0 0.0 rpy=0.0 0.0 0.0
- joint joint_6: axis 0 0 0 -> 0.0 0.0 0.0; limit lower=0 upper=0.03 effort=100 velocity=3 -> lower=0.0 upper=0.03 effort=100.0 velocity=3.0; origin xyz=0 0 0 rpy=0 0 0 -> xyz=0.0 0.0 0.0 rpy=0.0 0.0 0.0
- joint joint_7: axis 0 0 0 -> 0.0 0.0 0.0; limit lower=-0.03 upper=0 effort=100 velocity=3 -> lower=-0.03 upper=0.0 effort=100.0 velocity=3.0; origin xyz=0 0.8 0 rpy=3.1416 0 0 -> xyz=0.0 0.8 0.0 rpy=3.1416 0 0
